Commit message: revert to v5.1.0 with our params

File: zed_wrapper/urdf/zed_macro.urdf.xacro (robot description, xacro)
@@ -16,4 +16,5 @@
 -->
 <robot xmlns:xacro="http://wiki.ros.org/xacro">
+  <xacro:include filename="$(find zed_wrapper)/urdf/include/materials.urdf.xacro" />
   <xacro:property name="M_PI"     value="3.1415926535897931" />
   <!--
@@ -32,5 +33,4 @@
       <xacro:property name="optical_offset_x" value="-0.01" />
       <xacro:property name="mono" value="false" />
-      <xacro:property name="mat" value="0.8 0.8 0.8 1.0" />
     </xacro:if>
     <xacro:if value="${model == 'zedm'}">
@@ -42,5 +42,4 @@
       <xacro:property name="optical_offset_x" value="0.0" />
       <xacro:property name="mono" value="false" />
-      <xacro:property name="mat" value="0 0 0 1.0" />
     </xacro:if>
     <xacro:if value="${model == 'zed2'}">
@@ -52,5 +51,4 @@
       <xacro:property name="optical_offset_x" value="-0.01" />
       <xacro:property name="mono" value="false" />
-      <xacro:property name="mat" value="0.25 0.25 0.25 1.0" />
     </xacro:if>
     <xacro:if value="${model == 'zed2i'}">
@@ -62,5 +60,4 @@
       <xacro:property name="optical_offset_x" value="-0.01" />
       <xacro:property name="mono" value="false" />
-      <xacro:property name="mat" value="0.25 0.25 0.25 1.0" />
     </xacro:if>
     <xacro:if value="${model == 'zedx'}">
@@ -72,5 +69,4 @@
       <xacro:property name="optical_offset_x" value="-0.01" />
       <xacro:property name="mono" value="false" />
-      <xacro:property name="mat" value="0.25 0.25 0.25 1.0" />
     </xacro:if>
     <xacro:if value="${model == 'zedxhdr'}">
@@ -82,5 +78,4 @@
       <xacro:property name="optical_offset_x" value="-0.01" />
       <xacro:property name="mono" value="false" />
-      <xacro:property name="mat" value="0.25 0.25 0.25 1.0" />
     </xacro:if>
     <xacro:if value="${model == 'zedxm'}">
@@ -92,5 +87,4 @@
       <xacro:property name="optical_offset_x" value="-0.01" />
       <xacro:property name="mono" value="false" />
-      <xacro:property name="mat" value="0.25 0.25 0.25 1.0" />
     </xacro:if>
     <xacro:if value="${model == 'zedxhdrmini'}">
@@ -102,5 +96,4 @@
       <xacro:property name="optical_offset_x" value="-0.01" />
       <xacro:property name="mono" value="false" />
-      <xacro:property name="mat" value="0.25 0.25 0.25 1.0" />
     </xacro:if>
     <xacro:if value="${model == 'zedxhdrmax'}">
@@ -112,5 +105,4 @@
       <xacro:property name="optical_offset_x" value="-0.01" />
       <xacro:property name="mono" value="false" />
-      <xacro:property name="mat" value="0.25 0.25 0.25 1.0" />
     </xacro:if>
     <xacro:if value="${model == 'virtual'}">
@@ -122,5 +114,4 @@
       <xacro:property name="optical_offset_x" value="0.0" />
       <xacro:property name="mono" value="false" />
-      <xacro:property name="mat" value="0.25 0.25 0.25 1.0" />
     </xacro:if>
     <xacro:if value="${model == 'zedxonegs'}">
@@ -132,5 +123,4 @@
       <xacro:property name="optical_offset_x" value="0.0" />
       <xacro:property name="mono" value="true" />
-      <xacro:property name="mat" value="0.25 0.25 0.25 1.0" />
     </xacro:if>
     <xacro:if value="${model == 'zedxone4k'}">
@@ -142,5 +132,4 @@
       <xacro:property name="optical_offset_x" value="0.0" />
       <xacro:property name="mono" value="true" />
-      <xacro:property name="mat" value="0.25 0.25 0.25 1.0" />
     </xacro:if>
     <xacro:if value="${model == 'zedxonehdr'}">
@@ -152,5 +141,4 @@
       <xacro:property name="optical_offset_x" value="0.0" />
       <xacro:property name="mono" value="true" />
-      <xacro:property name="mat" value="0.25 0.25 0.25 1.0" />
     </xacro:if>
     <!-- Camera mounting point (the threaded screw hole in the bottom) -->
@@ -164,7 +152,5 @@
             <mesh filename="file://$(find zed_msgs)/meshes/${model}.stl"/>
           </geometry>
-            <material name="zed_mat">
-              <color rgba="${mat}"/>
-            </material>
+          <material name="${model}_mat" />
         </visual>
         <collision>
@@ -190,7 +176,5 @@
               <mesh filename="file://$(find zed_msgs)/meshes/${model}.stl"/>
             </geometry>
-            <material name="zed_mat">
-              <color rgba="${mat}"/>
-            </material>
+            <material name="${model}_mat" />
           </visual>
           <collision>
@@ -208,5 +192,5 @@
       </joint>
       <link name="${name}_left_camera_frame_optical"/>
-      <joint name="${name}_left_camera_joint_optical" type="fixed">
+      <joint name="${name}_left_camera_optical_joint" type="fixed">
         <origin xyz="0 0 0" rpy="-${M_PI/2} 0.0 -${M_PI/2}"/>
         <parent link="${name}_left_camera_frame"/>
@@ -221,7 +205,5 @@
               <mesh filename="file://$(find zed_msgs)/meshes/${model}.stl"/>
             </geometry>
-            <material name="zed_mat">
-              <color rgba="${mat}"/>
-            </material>
+            <material name="${model}_mat" />
           </visual>
           <collision>
@@ -239,5 +221,5 @@
       </joint>
       <link name="${name}_right_camera_frame_optical"/>
-      <joint name="${name}_right_camera_joint_optical" type="fixed">
+      <joint name="${name}_right_camera_optical_joint" type="fixed">
         <origin xyz="0 0 0" rpy="-${M_PI/2} 0.0 -${M_PI/2}"/>
         <parent link="${name}_right_camera_frame"/>
